File: Keyboard.kicad_pcb (KiCad board)
At the start: 2 copper layers, 290 x 190 mm, 391 parts, among them IC1 ATXMEGA128A4U-A, P1 USB_OTG, P2 CONN_PDI, SW1 SPST, SW10 Strg_L, SW11 F2, SW12 1, SW13 X, SW14 U, SW15 Ü, SW16 Wind_L, SW17 F3, SW18 2, SW19 V, SW2 SPST, SW20 I, SW21 Ö, SW22 Alt_L, SW23 M4_L, SW24 F4, SW25 3, SW26 L, SW27 A, SW28 Ä, SW29 M3_L, SW3 SPST, SW30 M5, SW31 F5, SW32 4, SW33 C, SW34 E, SW35 P, SW36 Back, SW37 enter, SW38 Drucken, SW39 O, SW4 SPST, SW40 Z, SW41 bottom_middle, SW42 F6, SW43 Rollen, SW44 5, SW45 W, SW46 Strg_M, SW47 grave, SW48 Entf, SW49 F7, SW5 SPST, SW50 Pause, SW51 6, SW52 K, SW53 mitte, SW54 aigu, SW55 M6, SW56 S, SW57 B, SW58 M4_R, SW59 leer, SW6 F1, SW60 F8, SW61 7, SW62 H, SW63 N, SW64 M, SW65 F9, SW66 8, SW67 G, SW68 R, SW69 komma, SW7 ESC, SW70 M3_R, SW71 F10, SW72 9, SW73 F, SW74 T, SW75 punkt, SW76 Wind_R, SW77 F11, SW78 0, SW79 Q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

Commit message: Add Gerbers sended to manufacturer
Other:
- rule pad_to_mask_clearance: 0.2 -> 0.05
- board text added: "Keyboard Rev: 0.1 09.03.2016"
Changed lines of the file:
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@@
     (area 64.924999 34.924999 355.075001 225.075001)
     (thickness 1.6)
-    (drawings 4)
-    (tracks 1460)
+    (drawings 5)
+    (tracks 1461)
     (zones 0)
     (modules 391)
@@
   (title_block
     (title Keyboard)
-    (date 2016-02-26)
+    (date 2016-03-09)
     (rev 0.1)
   )
@@
     (pad_size 0.6 0.6)
     (pad_drill 0.4)
-    (pad_to_mask_clearance 0.2)
+    (pad_to_mask_clearance 0.05)
     (aux_axis_origin 0 0)
     (visible_elements FFFFFF7F)
     (pcbplotparams
-      (layerselection 0x00030_80000001)
-      (usegerberextensions false)
+      (layerselection 0x010f0_80000001)
+      (usegerberextensions true)
       (excludeedgelayer true)
       (linewidth 0.100000)
@@
       (plotinvisibletext false)
       (padsonsilk false)
-      (subtractmaskfromsilk false)
+      (subtractmaskfromsilk true)
       (outputformat 1)
       (mirror false)
-      (drillshape 1)
+      (drillshape 0)
       (scaleselection 1)
-      (outputdirectory ""))
+      (outputdirectory Gerber/))
   )
   (net 0 "")
@@
     (descr "Through hole pin header")
     (tags "pin header")
-    (fp_text reference P2 (at 0 -5.1) (layer F.SilkS)
+    (fp_text reference P2 (at 1 -3) (layer F.SilkS)
       (effects (font (size 1 1) (thickness 0.15)))
     )
@@
     (descr "Mesurement Point, Square, Trough Hole,  DM 3mm, Drill 1.5mm,")
     (tags "Mesurement Point, Square, Trough Hole, DM 3mm, Drill 1.5mm,")
-    (fp_text reference W6 (at 0 -2.54) (layer F.SilkS)
+    (fp_text reference W6 (at 0 2.5) (layer F.Fab)
       (effects (font (size 1 1) (thickness 0.15)))
     )
-    (fp_text value C1 (at 0 3.81) (layer F.Fab)
+    (fp_text value C1 (at 0 -2.5) (layer F.SilkS)
       (effects (font (size 1 1) (thickness 0.15)))
     )
@@
     (descr "Mesurement Point, Square, Trough Hole,  DM 3mm, Drill 1.5mm,")
     (tags "Mesurement Point, Square, Trough Hole, DM 3mm, Drill 1.5mm,")
-    (fp_text reference W7 (at 0 -2.54) (layer F.SilkS)
+    (fp_text reference W7 (at 0 2.5) (layer F.Fab)
       (effects (font (size 1 1) (thickness 0.15)))
     )
-    (fp_text value C2 (at 0 3.81) (layer F.Fab)
+    (fp_text value C2 (at 0 -2.5) (layer F.SilkS)
       (effects (font (size 1 1) (thickness 0.15)))
     )
@@
     (descr "Mesurement Point, Square, Trough Hole,  DM 3mm, Drill 1.5mm,")
     (tags "Mesurement Point, Square, Trough Hole, DM 3mm, Drill 1.5mm,")
-    (fp_text reference W8 (at 0 -2.54) (layer F.SilkS)
+    (fp_text reference W8 (at 0 2.5) (layer F.Fab)
       (effects (font (size 1 1) (thickness 0.15)))
     )
-    (fp_text value C3 (at 0 3.81) (layer F.Fab)
+    (fp_text value C3 (at 0 -2.5) (layer F.SilkS)
       (effects (font (size 1 1) (thickness 0.15)))
     )
@@
     (descr "Mesurement Point, Square, Trough Hole,  DM 3mm, Drill 1.5mm,")
     (tags "Mesurement Point, Square, Trough Hole, DM 3mm, Drill 1.5mm,")
-    (fp_text reference W9 (at 0 -2.54) (layer F.SilkS)
+    (fp_text reference W9 (at 0 2.5) (layer F.Fab)
       (effects (font (size 1 1) (thickness 0.15)))
     )
-    (fp_text value C4 (at 0 3.81) (layer F.Fab)
+    (fp_text value C4 (at 0 -2.5) (layer F.SilkS)
       (effects (font (size 1 1) (thickness 0.15)))
     )
@@
     (descr "Mesurement Point, Square, Trough Hole,  DM 3mm, Drill 1.5mm,")
     (tags "Mesurement Point, Square, Trough Hole, DM 3mm, Drill 1.5mm,")
-    (fp_text reference W10 (at 0 -2.54) (layer F.SilkS)
+    (fp_text reference W10 (at 0 2.5) (layer F.Fab)
       (effects (font (size 1 1) (thickness 0.15)))
     )
-    (fp_text value C5 (at 0 3.81) (layer F.Fab)
+    (fp_text value C5 (at 0 -2.5) (layer F.SilkS)
       (effects (font (size 1 1) (thickness 0.15)))
     )
@@
     (descr "Mesurement Point, Square, Trough Hole,  DM 3mm, Drill 1.5mm,")
     (tags "Mesurement Point, Square, Trough Hole, DM 3mm, Drill 1.5mm,")
-    (fp_text reference W11 (at 0 -2.54) (layer F.SilkS)
+    (fp_text reference W11 (at 0 2.5) (layer F.Fab)
       (effects (font (size 1 1) (thickness 0.15)))
     )
-    (fp_text value C6 (at 0 3.81) (layer F.Fab)
+    (fp_text value C6 (at 0 -2.5) (layer F.SilkS)
       (effects (font (size 1 1) (thickness 0.15)))
     )
@@
     (descr "Mesurement Point, Square, Trough Hole,  DM 3mm, Drill 1.5mm,")
     (tags "Mesurement Point, Square, Trough Hole, DM 3mm, Drill 1.5mm,")
-    (fp_text reference W12 (at 0 -2.54) (layer F.SilkS)
+    (fp_text reference W12 (at 0 2.5) (layer F.Fab)
       (effects (font (size 1 1) (thickness 0.15)))
     )
-    (fp_text value C7 (at 0 3.81) (layer F.Fab)
+    (fp_text value C7 (at 0 -2.5) (layer F.SilkS)
       (effects (font (size 1 1) (thickness 0.15)))
     )
@@
     (descr "Mesurement Point, Square, Trough Hole,  DM 3mm, Drill 1.5mm,")
     (tags "Mesurement Point, Square, Trough Hole, DM 3mm, Drill 1.5mm,")
-    (fp_text reference W13 (at 0 -2.54) (layer F.SilkS)
+    (fp_text reference W13 (at 0 2.5) (layer F.Fab)
       (effects (font (size 1 1) (thickness 0.15)))
     )
-    (fp_text value C8 (at 0 3.81) (layer F.Fab)
+    (fp_text value C8 (at 0 -2.5) (layer F.SilkS)
       (effects (font (size 1 1) (thickness 0.15)))
     )
@@
     (descr "Mesurement Point, Square, Trough Hole,  DM 3mm, Drill 1.5mm,")
     (tags "Mesurement Point, Square, Trough Hole, DM 3mm, Drill 1.5mm,")
-    (fp_text reference W14 (at 0 -2.54) (layer F.SilkS)
+    (fp_text reference W14 (at 0 2.5) (layer F.Fab)
       (effects (font (size 1 1) (thickness 0.15)))
     )
-    (fp_text value C9 (at 0 3.81) (layer F.Fab)
+    (fp_text value C9 (at 0 -2.5) (layer F.SilkS)
       (effects (font (size 1 1) (thickness 0.15)))
     )
@@
     (descr "Mesurement Point, Square, Trough Hole,  DM 3mm, Drill 1.5mm,")
     (tags "Mesurement Point, Square, Trough Hole, DM 3mm, Drill 1.5mm,")
-    (fp_text reference W15 (at 0 -2.54) (layer F.SilkS)
+    (fp_text reference W15 (at 0 2.5) (layer F.Fab)
       (effects (font (size 1 1) (thickness 0.15)))
     )
-    (fp_text value C10 (at 0 3.81) (layer F.Fab)
+    (fp_text value C10 (at 0 -2.5) (layer F.SilkS)
       (effects (font (size 1 1) (thickness 0.15)))
     )
@@
     (descr "Mesurement Point, Square, Trough Hole,  DM 3mm, Drill 1.5mm,")
     (tags "Mesurement Point, Square, Trough Hole, DM 3mm, Drill 1.5mm,")
-    (fp_text reference W16 (at 0 -2.54) (layer F.SilkS)
+    (fp_text reference W16 (at 0 2.5) (layer F.Fab)
       (effects (font (size 1 1) (thickness 0.15)))
     )
-    (fp_text value C11 (at 0 3.81) (layer F.Fab)
+    (fp_text value C11 (at 0 -2.5) (layer F.SilkS)
       (effects (font (size 1 1) (thickness 0.15)))
     )
@@
     (descr "Mesurement Point, Square, Trough Hole,  DM 3mm, Drill 1.5mm,")
     (tags "Mesurement Point, Square, Trough Hole, DM 3mm, Drill 1.5mm,")
-    (fp_text reference W17 (at 0 -2.54) (layer F.SilkS)
+    (fp_text reference W17 (at 0 2.5) (layer F.Fab)
       (effects (font (size 1 1) (thickness 0.15)))
     )
-    (fp_text value C12 (at 0 3.81) (layer F.Fab)
+    (fp_text value C12 (at 0 -2.5) (layer F.SilkS)
       (effects (font (size 1 1) (thickness 0.15)))
     )
@@
       (net 2 GND) (zone_connect 2))
   )
+  (gr_text "Keyboard\nRev: 0.1\n09.03.2016" (at 85 205.5) (layer B.SilkS)
+    (effects (font (size 1.5 1.5) (thickness 0.3)) (justify mirror))
+  )
   (gr_line (start 65 225) (end 355 225) (angle 90) (layer Edge.Cuts) (width 0.15))
   (gr_line (start 65 35) (end 65 225) (angle 90) (layer Edge.Cuts) (width 0.15))
@@
   (segment (start 277.354332 74.596428) (end 277.50076 74.45) (width 0.3) (layer B.Cu) (net 82))
   (segment (start 277.256248 79.45) (end 277.354332 79.351916) (width 0.3) (layer B.Cu) (net 82))
+  (segment (start 275.50178 73.5) (end 275 74.00178) (width 0.3) (layer B.Cu) (net 83))
+  (segment (start 275 74.00178) (end 275 85.792878) (width 0.3) (layer B.Cu) (net 83))
+  (segment (start 279.5 90.292878) (end 279.5 102.792878) (width 0.3) (layer B.Cu) (net 83))
+  (segment (start 275 85.792878) (end 279.5 90.292878) (width 0.3) (layer B.Cu) (net 83))
+  (segment (start 279.5 102.792878) (end 285.00178 108.294658) (width 0.3) (layer B.Cu) (net 83))
+  (segment (start 285.00178 108.294658) (end 285.00178 110.29995) (width 0.3) (layer B.Cu) (net 83))
+  (segment (start 285.00178 110.29995) (end 285.00178 111) (width 0.3) (layer B.Cu) (net 83))
   (segment (start 295.00178 147) (end 295.00178 145.294658) (width 0.3) (layer B.Cu) (net 83))
   (segment (start 295.00178 145.294658) (end 289 139.292878) (width 0.3) (layer B.Cu) (net 83))
@@
   (segment (start 290 176.5) (end 290 184) (width 0.3) (layer B.Cu) (net 83))
   (segment (start 287 190.1) (end 288.7 191.8) (width 0.3) (layer B.Cu) (net 83))
-  (segment (start 279.5 102.792878) (end 285.00178 108.294658) (width 0.3) (layer B.Cu) (net 83))
-  (segment (start 275.50178 86.294658) (end 279.5 90.292878) (width 0.3) (layer B.Cu) (net 83))
-  (segment (start 275.50178 73.5) (end 275.50178 86.294658) (width 0.3) (layer B.Cu) (net 83))
-  (segment (start 279.5 90.292878) (end 279.5 102.792878) (width 0.3) (layer B.Cu) (net 83))
-  (segment (start 285.00178 108.294658) (end 285.00178 110.29995) (width 0.3) (layer B.Cu) (net 83))
-  (segment (start 285.00178 110.29995) (end 285.00178 111) (width 0.3) (layer B.Cu) (net 83))
   (segment (start 287.00076 110.05) (end 287.00076 104.50076) (width 0.3) (layer B.Cu) (net 84))
   (segment (start 287.00076 104.50076) (end 283.476401 100.976401) (width 0.3) (layer B.Cu) (net 84))
